File: Circuit Design/nixie-panel/nixie-panel.kicad_sch (KiCad schematic)
At the start: 8 parts, among them J1 Conn_01x06, J2 Conn_01x06

Commit message: the routing and fine touching is done. Ready for production
Parts:
- added C1, C10, C4, C7: 1uF, CoF_Capacitor:C-0402, symbol CoE_Capacitor:1uF
- added C11, C12, C2, C3, C5, C6, C8, C9: 100nF, CoF_Capacitor:C-0402, symbol CoE_Capacitor:100nF
Connections:
- net +3V3: now also J1.4 (Pin_4), J2.4 (Pin_4), C1.1, C10.1, C11.1, C12.1, C2.1, C3.1, C4.1, C5.1, C6.1, C7.1, C8.1, C9.1; no longer J1.6 (Pin_6), J2.6 (Pin_6)
- net GND: now also C1.2, C10.2, C11.2, C12.2, C2.2, C3.2, C4.2, C5.2, C6.2, C7.2, C8.2, C9.2
- net I2C0-SCL: now also J1.5 (Pin_5); no longer J1.3 (Pin_3)
- net I2C0-SDA: now also J1.3 (Pin_3); no longer J1.4 (Pin_4)
- net I2C1-SDA: now also J2.5 (Pin_5); no longer J2.4 (Pin_4)
- net LightSense2: now also J1.6 (Pin_6); no longer J1.5 (Pin_5)
Other:
- moved on the sheet: J2
